File: buzzcar_main/buzzcar_main.kicad_sch (KiCad schematic)
At the start: 44 parts, among them J1 9V Battery Cap, J2 5V Buck, J3 3.3V Buck, J4 Motor_A, J5 Motor_B, J6 Video GME12864, J7 Audio Amp PAM8904, J8 8Ω Speaker, SW1 Main Power, SW2 SW_Push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

Commit message: PCB Layout v0.1 done
Parts:
- removed D1: LED_C, symbol Device:LED
- removed D2: LED_B, symbol Device:LED
- removed D3: LED_A, symbol Device:LED
- removed R10, R11, R12: 47, symbol Device:R_US
- removed R4, R5, R6: R_Photo, symbol Device:R_Photo
- removed R7, R8, R9: 3k, Resistor_THT:R_Axial_DIN0207_L6.3mm_D2.5mm_P10.16mm_Horizontal, symbol Device:R_US
- removed TP12, TP13: TestPoint, symbol Connector:TestPoint
- added J10: Sensor_B, Connector_PinHeader_2.54mm:PinHeader_1x04_P2.54mm_Vertical, symbol Connector:Conn_01x04_Socket
- added J11: Sensor_A, Connector_PinHeader_2.54mm:PinHeader_1x04_P2.54mm_Vertical, symbol Connector:Conn_01x04_Socket
- added J9: Sensor_C, Connector_PinHeader_2.54mm:PinHeader_1x04_P2.54mm_Vertical, symbol Connector:Conn_01x04_Socket
- added TP3: 5v0, TestPoint:TestPoint_Loop_D2.60mm_Drill1.6mm_Beaded, symbol Connector:TestPoint
- added TP4: 3v3, TestPoint:TestPoint_Loop_D2.60mm_Drill1.6mm_Beaded, symbol Connector:TestPoint
- D1: renamed from D4; footprint (none) -> LED_THT:LED_D3.0mm
- H1, H2, H3, H4: footprint (none) -> MountingHole:MountingHole_3mm
- J1, J4, J5: footprint (none) -> Connector_PinHeader_2.54mm:PinHeader_1x02_P2.54mm_Vertical
- R4: renamed from R13; footprint (none) -> Resistor_THT:R_Axial_DIN0207_L6.3mm_D2.5mm_P10.16mm_Horizontal
- SW2: value SW_Push -> Motion_Sw; footprint (none) -> Connector_PinHeader_2.54mm:PinHeader_1x02_P2.54mm_Vertical
- TP10: renamed from TP9; value TestPoint -> motion_sw; footprint (none) -> TestPoint:TestPoint_Loop_D2.60mm_Drill1.6mm_Beaded
- TP5: renamed from TP6; value TestPoint -> motion_9v0; footprint (none) -> TestPoint:TestPoint_Loop_D2.60mm_Drill1.6mm_Beaded
- TP6: renamed from TP7; value TestPoint -> motion_3v3; footprint (none) -> TestPoint:TestPoint_Loop_D2.60mm_Drill1.6mm_Beaded
- TP7: renamed from TP8; value TestPoint -> control_5v0; footprint (none) -> TestPoint:TestPoint_Loop_D2.60mm_Drill1.6mm_Beaded
- TP8: renamed from TP10; value TestPoint -> control_gnd; footprint (none) -> TestPoint:TestPoint_Loop_D2.60mm_Drill1.6mm_Beaded
- TP9: renamed from TP11; value TestPoint -> control_gnd2; footprint (none) -> TestPoint:TestPoint_Loop_D2.60mm_Drill1.6mm_Beaded
Connections:
- net +3.3V: now also J10.2 (Pin_2), J11.2 (Pin_2), J9.2 (Pin_2), TP4.1
- net +5V: now also J10.1 (Pin_1), J11.1 (Pin_1), J9.1 (Pin_1), TP3.1
- net GND: now also J10.3 (Pin_3), J11.3 (Pin_3), J9.3 (Pin_3)
- net din_a renamed sig_a
- net sig_a: now also J11.4 (Pin_4)
- net din_b renamed sig_b
- net sig_b: now also J10.4 (Pin_4)
- net din_c renamed sig_c
- net sig_c: now also J9.4 (Pin_4)
Other:
- moved on the sheet: D1, J2, J3, R1, R2, R4, TP1, TP2, TP9, U2

Commit message: PCB Layout v0.2 done - silkscreen errors left
Parts:
- added J12: Safety, Connector_PinHeader_2.54mm:PinHeader_1x05_P2.54mm_Vertical, symbol Connector:Conn_01x05_Socket
Connections:
- net at U1.3 (GPIO4/MTMS): now also J12.5 (Pin_5)
- net at U1.4 (GPIO5/MTDI): now also J12.4 (Pin_4)
- net at U1.5 (GPIO6): now also J12.3 (Pin_3)
- net at U1.6 (GPIO7): now also J12.2 (Pin_2)
- net at U1.7 (GPIO0): now also J12.1 (Pin_1)
- no-connect marks 19 -> 14
Changed lines of the file:
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@@
 	)
 	(no_connect
-		(at 194.31 96.52)
-	)
-	(no_connect
-		(at 194.31 93.98)
-	)
-	(no_connect
 		(at 69.85 100.33)
 	)
@@
 	)
 	(no_connect
-		(at 194.31 99.06)
-	)
-	(no_connect
 		(at 245.11 88.9)
 	)
@@
 	)
 	(no_connect
-		(at 194.31 88.9)
-	)
-	(no_connect
-		(at 194.31 91.44)
-	)
-	(no_connect
 		(at 245.11 109.22)
 	)
@@
 	(wire
 		(pts
+			(xy 190.5 96.52) (xy 194.31 96.52)
+		)
+		(stroke
+			(width 0)
+			(type default)
+		)
+	)
+	(wire
+		(pts
 			(xy 76.2 157.48) (xy 77.47 157.48)
 		)
@@
 	(wire
 		(pts
+			(xy 190.5 88.9) (xy 194.31 88.9)
+		)
+		(stroke
+			(width 0)
+			(type default)
+		)
+	)
+	(wire
+		(pts
 			(xy 105.41 90.17) (xy 110.49 90.17)
 		)
@@
 	(wire
 		(pts
+			(xy 190.5 91.44) (xy 194.31 91.44)
+		)
+		(stroke
+			(width 0)
+			(type default)
+		)
+	)
+	(wire
+		(pts
 			(xy 168.91 109.22) (xy 168.91 116.84)
 		)
@@
 	(wire
 		(pts
+			(xy 190.5 93.98) (xy 194.31 93.98)
+		)
+		(stroke
+			(width 0)
+			(type default)
+		)
+	)
+	(wire
+		(pts
 			(xy 30.48 82.55) (xy 33.02 82.55)
 		)
@@
 	(wire
 		(pts
+			(xy 190.5 99.06) (xy 194.31 99.06)
+		)
+		(stroke
+			(width 0)
+			(type default)
+		)
+	)
+	(wire
+		(pts
 			(xy 134.62 184.15) (xy 138.43 184.15)
 		)
@@
 					(unit 1)
 				)
+			)
+		)
+	)
+	(symbol
+		(lib_id "Connector:Conn_01x05_Socket")
+		(at 185.42 93.98 180)
+		(unit 1)
+		(exclude_from_sim no)
+		(in_bom yes)
+		(on_board yes)
+		(dnp no)
+		(property "Reference" "J12"
+			(at 181.864 93.726 0)
+			(effects
+				(font
+					(size 1.27 1.27)
+				)
+			)
+		)
+		(property "Value" "Safety"
+			(at 181.864 95.504 0)
+			(effects
+				(font
+					(size 1.27 1.27)
+				)
+			)
+		)
+		(property "Footprint" "Connector_PinHeader_2.54mm:PinHeader_1x05_P2.54mm_Vertical"
+			(at 185.42 93.98 0)
+			(effects
+				(font
+					(size 1.27 1.27)
+				)
+				(hide yes)
+			)
+		)
+		(property "Datasheet" "~"
+			(at 185.42 93.98 0)
+			(effects
+				(font
+					(size 1.27 1.27)
+				)
+				(hide yes)
+			)
+		)
+		(property "Description" "Generic connector, single row, 01x05, script generated"
+			(at 185.42 93.98 0)
+			(effects
+				(font
+					(size 1.27 1.27)
+				)
+				(hide yes)
+			)
+		)
+		(pin "5"
+		)
+		(pin "4"
+		)
+		(pin "2"
+		)
+		(pin "3"
+		)
+		(pin "1"
+		)
+		(instances
+			(project ""
+				(path "/0725cd7b-8909-454f-8cd3-1584cffd5410"
+					(reference "J12")
+					(unit 1)
+				)
